Commit message: Convert URDF package to ROS 2 and fix mesh paths

File: arm_7dof_urdf/urdf/arm_7dof_urdf.urdf (robot description, URDF)
Before this commit: robot 7dof-arm-urdf, 8 links, 7 joints
Links:
- link base: geometry collision mesh filename=package://arm_7dof_urdf/meshes/base.STL; visual mesh filename=package://arm_7dof_urdf/meshes/base.STL
- link link_1: geometry collision mesh filename=package://arm_7dof_urdf/meshes/link_1.STL; visual mesh filename=package://arm_7dof_urdf/meshes/link_1.STL
- link link_2: geometry collision mesh filename=package://arm_7dof_urdf/meshes/link_2.STL; visual mesh filename=package://arm_7dof_urdf/meshes/link_2.STL
- link link_3: geometry collision mesh filename=package://arm_7dof_urdf/meshes/link_3.STL; visual mesh filename=package://arm_7dof_urdf/meshes/link_3.STL
- link link_4: geometry collision mesh filename=package://arm_7dof_urdf/meshes/link_4.STL; visual mesh filename=package://arm_7dof_urdf/meshes/link_4.STL
- link link_5: geometry collision mesh filename=package://arm_7dof_urdf/meshes/link_5.STL; visual mesh filename=package://arm_7dof_urdf/meshes/link_5.STL
- link link_6: geometry collision mesh filename=package://arm_7dof_urdf/meshes/link_6.STL; visual mesh filename=package://arm_7dof_urdf/meshes/link_6.STL
- link link_7: geometry collision mesh filename=package://arm_7dof_urdf/meshes/link_7.STL; visual mesh filename=package://arm_7dof_urdf/meshes/link_7.STL
Joints:
- joint joint_1: limit lower=0 upper=0 effort=0 velocity=0 -> lower=-3.14159 upper=3.14159 effort=10 velocity=1.0
- joint joint_2: limit lower=0 upper=0 effort=0 velocity=0 -> lower=-3.14159 upper=3.14159 effort=10 velocity=1.0
- joint joint_3: limit lower=0 upper=0 effort=0 velocity=0 -> lower=-3.14159 upper=3.14159 effort=10 velocity=1.0
- joint joint_4: limit lower=0 upper=0 effort=0 velocity=0 -> lower=-3.14159 upper=3.14159 effort=10 velocity=1.0
- joint joint_5: limit lower=0 upper=0 effort=0 velocity=0 -> lower=-3.14159 upper=3.14159 effort=10 velocity=1.0
- joint joint_6: limit lower=0 upper=0 effort=0 velocity=0 -> lower=-3.14159 upper=3.14159 effort=10 velocity=1.0
- joint joint_7: limit lower=0 upper=0 effort=0 velocity=0 -> lower=-3.14159 upper=3.14159 effort=10 velocity=1.0

Commit message: Range of joint 2, 4, 6 adjusted to +/- 90 degrees

File: arm_7dof_urdf/urdf/arm_7dof_urdf.urdf (robot description, URDF)
Before this commit: robot arm_7dof_urdf, 8 links, 7 joints
Joints:
- joint joint_2: limit lower=-3.14159 upper=3.14159 effort=10 velocity=1.0 -> lower=-1.5708 upper=1.5708 effort=10 velocity=1.0
- joint joint_4: limit lower=-3.14159 upper=3.14159 effort=10 velocity=1.0 -> lower=-1.5708 upper=1.5708 effort=10 velocity=1.0
- joint joint_6: limit lower=-3.14159 upper=3.14159 effort=10 velocity=1.0 -> lower=-1.5708 upper=1.5708 effort=10 velocity=1.0
