Commit message: Rename folder

File: arm_7dof/urdf/arm_7dof.urdf (robot description, URDF)
Before this commit: robot arm_7dof_urdf, 8 links, 7 joints
Links:
- link base: geometry collision mesh filename=package://arm_7dof/meshes/base.STL; visual mesh filename=package://arm_7dof/meshes/base.STL
- link link_1: geometry collision mesh filename=package://arm_7dof/meshes/link_1.STL; visual mesh filename=package://arm_7dof/meshes/link_1.STL
- link link_2: geometry collision mesh filename=package://arm_7dof/meshes/link_2.STL; visual mesh filename=package://arm_7dof/meshes/link_2.STL
- link link_3: geometry collision mesh filename=package://arm_7dof/meshes/link_3.STL; visual mesh filename=package://arm_7dof/meshes/link_3.STL
- link link_4: geometry collision mesh filename=package://arm_7dof/meshes/link_4.STL; visual mesh filename=package://arm_7dof/meshes/link_4.STL
- link link_5: geometry collision mesh filename=package://arm_7dof/meshes/link_5.STL; visual mesh filename=package://arm_7dof/meshes/link_5.STL
- link link_6: geometry collision mesh filename=package://arm_7dof/meshes/link_6.STL; visual mesh filename=package://arm_7dof/meshes/link_6.STL
- link link_7: geometry collision mesh filename=package://arm_7dof/meshes/link_7.STL; visual mesh filename=package://arm_7dof/meshes/link_7.STL
